File: PCB/ostc_v2/ostc_v2.brd (EAGLE design)
At the start: 31.5 x 54.8 mm, 13 parts, among them IC3 150-10-640-00-001000, U1 ICO-640-SGG, U2 XC9536XL-10CSG48I, U3 IS62C256AL-45TLI, U4 LP5912Q3.3DRVRQ1, X1 505567-0651

Commit message: Modified schematics & boards
Parts:
- added X2: 505567-0251, con-molex:53261-02
- renumbered IC3 to X3
Connections:
- new net N$47: U2.E3, U3.9
- new net N$48: U2.F6, U3.10
- new net N$49: U2.G4, U3.22
- new net N$50: U2.F4, U3.20
- new net N$51: U2.F2, U3.27
- net GND: now also X2.2
- net N$45: now also X2.1

Commit message: Updated PCB files
Parts:
- removed R2: 2k, resistor:R0805
- R1: value 4k -> 4k7
- moved X2 10.0 mm to (28.8, 48.2)
Connections:
- removed net N$46: R2.1, S1.2
- net GND: now also S1.2, X2.1; no longer R2.2, X2.2
- net N$45: now also X2.2; no longer X2.1
Routing:
- net N$46: track 9.04 -> 0.00 mm, vias 1 -> 0
- net +3.3V: track 72.8 -> 64.9 mm
- net N$45: track 66.8 -> 59.6 mm
- net N$58: track 72.8 -> 69.6 mm
- net N$57: track 79.1 -> 81.8 mm

Commit message: Corrected PCB
Routing:
- net N$49: track 0.00 -> 36.1 mm, vias 0 -> 4
- net N$51: track 0.00 -> 27.9 mm, vias 0 -> 3
- net N$48: track 0.00 -> 13.9 mm, vias 0 -> 2
- net N$47: track 0.00 -> 13.8 mm, vias 0 -> 2
- net N$50: track 0.00 -> 13.2 mm, vias 0 -> 2
- net N$38: track 28.5 -> 35.6 mm
- net +3.3V: track 64.9 -> 71.0 mm, vias 0 -> 4
- net +5V: track 22.5 -> 27.5 mm, vias 2 -> 3
- net GND: track 27.1 -> 32.1 mm, vias 12 -> 19
- net N$37: track 28.1 -> 31.1 mm
- net N$43: track 33.9 -> 35.3 mm
- net N$44: track 23.6 -> 24.8 mm
- net N$57: track 81.8 -> 81.1 mm
Other:
- board text added: "6502"
- board text added: "External Switch"

Commit message: Updated PCB
Routing:
- net N$38: track 35.6 -> 32.1 mm
- net N$57: track 81.1 -> 79.1 mm
Changed lines of the file:
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@@
 Layout by zchap40</text>
 <text x="14.95" y="1.95" size="1.016" layer="25" font="vector" ratio="18" align="bottom-right">6502</text>
-<text x="31.1" y="52.45" size="0.6096" layer="26" font="vector" ratio="18" rot="MR0">External
+<text x="31.1" y="52.65" size="0.6096" layer="26" font="vector" ratio="18" rot="MR0">External
 Switch</text>
 </plain>
@@
 </element>
 <element name="R1" library="resistor" package="R0805" value="4k7" x="25.44" y="40.54" smashed="yes" rot="MR180">
-<attribute name="NAME" x="22.726" y="39.8" size="1.016" layer="26" font="vector" ratio="18" rot="MR90"/>
-<attribute name="VALUE" x="27.174" y="39.778" size="0.6096" layer="28" font="vector" ratio="18" rot="MR90"/>
+<attribute name="NAME" x="28.424" y="41.7" size="1.016" layer="26" font="vector" ratio="18" rot="MR270"/>
+<attribute name="VALUE" x="25.022" y="41.724" size="0.6096" layer="28" font="vector" ratio="18" rot="MR0"/>
 </element>
 <element name="C1" library="resistor" package="C1206K" value="10u" x="11.56" y="49.62" smashed="yes" rot="MR0">
@@
 <wire x1="9.21" y1="30.69" x2="9.2" y2="31.8375" width="0.3048" layer="16"/>
 <via x="9.2" y="31.8375" extent="1-16" drill="0.25" diameter="0.45"/>
-<wire x1="9.2" y1="31.8375" x2="9.65" y2="32.3" width="0.3048" layer="1"/>
-<wire x1="9.65" y1="32.3" x2="13.95" y2="32.3" width="0.3048" layer="1"/>
-<wire x1="13.95" y1="32.3" x2="14.4" y2="32.75" width="0.3048" layer="1"/>
-<wire x1="14.4" y1="32.75" x2="14.4" y2="43" width="0.3048" layer="1"/>
-<wire x1="14.4" y1="43" x2="14.9" y2="43.45" width="0.3048" layer="1"/>
-<wire x1="14.9" y1="43.45" x2="17.76" y2="43.45" width="0.3048" layer="1"/>
+<wire x1="9.2" y1="31.8375" x2="9.2" y2="32.8" width="0.3048" layer="1"/>
+<wire x1="9.2" y1="32.8" x2="9.5" y2="33.1" width="0.3048" layer="1"/>
+<wire x1="9.5" y1="33.1" x2="13.05" y2="33.1" width="0.3048" layer="1"/>
+<wire x1="13.05" y1="33.1" x2="13.55" y2="33.7" width="0.3048" layer="1"/>
+<wire x1="13.55" y1="33.7" x2="13.55" y2="43.15" width="0.3048" layer="1"/>
+<wire x1="13.55" y1="43.15" x2="13.9" y2="43.45" width="0.3048" layer="1"/>
+<wire x1="13.9" y1="43.45" x2="17.76" y2="43.45" width="0.3048" layer="1"/>
 <wire x1="17.76" y1="43.45" x2="17.78" y2="43.43" width="0.3048" layer="1"/>
 </signal>
@@
 <contactref element="U3" pad="12"/>
 <contactref element="U2" pad="E5"/>
-<wire x1="9" y1="29.3" x2="9" y2="22.75" width="0.3048" layer="15"/>
+<wire x1="9" y1="28.05" x2="9" y2="22.75" width="0.3048" layer="15"/>
 <wire x1="9" y1="22.75" x2="9.1" y2="22.65" width="0.3048" layer="15"/>
 <wire x1="9.1" y1="22.65" x2="10.3" y2="22.65" width="0.3048" layer="15"/>
@@
 <via x="10.325" y="17.3375" extent="1-16" drill="0.25" diameter="0.45"/>
 <wire x1="10.325" y1="17.3375" x2="10.325" y2="15.91" width="0.3048" layer="16"/>
-<wire x1="12.85" y1="28.55" x2="12.85" y2="29.7" width="0.3048" layer="2"/>
-<wire x1="12.85" y1="29.7" x2="13.1" y2="29.85" width="0.3048" layer="2"/>
-<wire x1="13.1" y1="29.85" x2="15.3" y2="29.85" width="0.3048" layer="2"/>
-<wire x1="15.3" y1="29.85" x2="15.55" y2="30.1" width="0.3048" layer="2"/>
-<wire x1="15.55" y1="30.1" x2="15.55" y2="31.65" width="0.3048" layer="2"/>
-<wire x1="15.55" y1="31.65" x2="15.9" y2="32" width="0.3048" layer="2"/>
-<wire x1="15.9" y1="32" x2="19.82" y2="32" width="0.3048" layer="2"/>
+<wire x1="11.75" y1="27.55" x2="13.95" y2="29.75" width="0.3048" layer="2"/>
+<wire x1="13.95" y1="29.75" x2="16.1" y2="29.8" width="0.3048" layer="2"/>
+<wire x1="16.1" y1="29.8" x2="16.4" y2="30.1" width="0.3048" layer="2"/>
+<wire x1="16.4" y1="30.1" x2="16.4" y2="31.7" width="0.3048" layer="2"/>
+<wire x1="16.4" y1="31.7" x2="16.85" y2="32" width="0.3048" layer="2"/>
+<wire x1="16.85" y1="32" x2="19.82" y2="32" width="0.3048" layer="2"/>
 <wire x1="19.82" y1="32" x2="21.09" y2="30.73" width="0.3048" layer="2"/>
 <wire x1="10.81" y1="26.21" x2="10.81" y2="26.24" width="0.125" layer="16"/>
 <wire x1="10.81" y1="26.24" x2="10.4" y2="26.6" width="0.125" layer="16"/>
 <via x="10.4" y="26.6" extent="1-16" drill="0.25" diameter="0.45"/>
-<wire x1="10.4" y1="26.6" x2="11.6" y2="27.45" width="0.3048" layer="15"/>
-<wire x1="11.6" y1="27.45" x2="11.6" y2="27.55" width="0.3048" layer="15"/>
-<wire x1="11.6" y1="27.55" x2="10.7" y2="28.45" width="0.3048" layer="15"/>
-<wire x1="10.7" y1="28.45" x2="10.7" y2="29.05" width="0.3048" layer="15"/>
-<wire x1="10.7" y1="29.05" x2="10.45" y2="29.3" width="0.3048" layer="15"/>
-<wire x1="10.45" y1="29.3" x2="9" y2="29.3" width="0.3048" layer="15"/>
-<wire x1="12.85" y1="28.55" x2="11.75" y2="27.55" width="0.3048" layer="2"/>
+<wire x1="10.4" y1="26.6" x2="11.05" y2="27.1" width="0.3048" layer="15"/>
+<wire x1="11.05" y1="27.1" x2="11.05" y2="27.7" width="0.3048" layer="15"/>
+<wire x1="11.05" y1="27.7" x2="10.7" y2="28.05" width="0.3048" layer="15"/>
+<wire x1="10.7" y1="28.05" x2="9" y2="28.05" width="0.3048" layer="15"/>
 <wire x1="11.75" y1="27.55" x2="10.4" y2="26.6" width="0.3048" layer="2"/>
 </signal>
@@
 <wire x1="29.25" y1="32.4" x2="24.7" y2="32.4" width="0.3048" layer="15"/>
 <wire x1="24.7" y1="32.4" x2="24.35" y2="32.75" width="0.3048" layer="15"/>
-<wire x1="24.35" y1="32.75" x2="24.35" y2="50.35" width="0.3048" layer="15"/>
-<wire x1="24.35" y1="50.35" x2="24.5" y2="50.5" width="0.3048" layer="15"/>
-<wire x1="24.5" y1="50.5" x2="25.5" y2="50.5" width="0.3048" layer="15"/>
-<wire x1="25.5" y1="50.5" x2="25.75" y2="50.75" width="0.3048" layer="15"/>
-<wire x1="25.75" y1="50.75" x2="25.75" y2="52.85" width="0.3048" layer="15"/>
-<wire x1="25.75" y1="52.85" x2="25.45" y2="53.15" width="0.15" layer="15"/>
-<wire x1="25.45" y1="53.15" x2="14.55" y2="53.15" width="0.15" layer="15"/>
+<wire x1="24.35" y1="32.75" x2="24.35" y2="51.65" width="0.3048" layer="15"/>
+<wire x1="24.35" y1="51.65" x2="24.8" y2="51.65" width="0.3048" layer="15"/>
+<wire x1="24.8" y1="51.65" x2="25.1" y2="51.9" width="0.3048" layer="15"/>
+<wire x1="25.1" y1="51.9" x2="25.1" y2="52.9" width="0.3048" layer="15"/>
+<wire x1="25.1" y1="52.9" x2="24.9" y2="53.15" width="0.15" layer="15"/>
+<wire x1="24.9" y1="53.15" x2="14.55" y2="53.15" width="0.15" layer="15"/>
 <wire x1="14.55" y1="53.15" x2="8.2" y2="53.15" width="0.3048" layer="15"/>
 <wire x1="8.2" y1="53.15" x2="7.9" y2="52.9" width="0.3048" layer="15"/>
 <wire x1="7.9" y1="52.9" x2="7.9" y2="30.7" width="0.3048" layer="15"/>
 <wire x1="7.9" y1="30.7" x2="8.45" y2="30.2" width="0.3048" layer="15"/>
-<wire x1="8.45" y1="30.2" x2="8.45" y2="27.8" width="0.3048" layer="15"/>
-<wire x1="8.45" y1="27.8" x2="7.8" y2="27" width="0.3048" layer="15"/>
-<wire x1="7.8" y1="27" x2="7.8" y2="22.55" width="0.3048" layer="15"/>
-<wire x1="7.8" y1="22.55" x2="8.0375" y2="22.325" width="0.3048" layer="15"/>
-<wire x1="8.0375" y1="22.325" x2="8.625" y2="22.325" width="0.3048" layer="15"/>
+<wire x1="8.45" y1="30.2" x2="8.45" y2="22.5125" width="0.3048" layer="15"/>
+<wire x1="8.45" y1="22.5125" x2="8.625" y2="22.325" width="0.3048" layer="15"/>
 <via x="8.625" y="22.325" extent="1-16" drill="0.25" diameter="0.5"/>
 <wire x1="8.625" y1="22.325" x2="8.625" y2="23.8" width="0.15" layer="16"/>
@@
 <wire x1="9.5" y1="14.7" x2="9.55" y2="14.75" width="0.3048" layer="15"/>
 <via x="9.55" y="14.75" extent="1-16" drill="0.25"/>
-<wire x1="9.55" y1="14.75" x2="7.65" y2="14.75" width="0.3048" layer="2"/>
-<wire x1="7.65" y1="14.75" x2="7.4" y2="15" width="0.3048" layer="2"/>
-<wire x1="7.4" y1="15" x2="7.4" y2="26.75" width="0.3048" layer="2"/>
+<wire x1="9.55" y1="14.75" x2="9.55" y2="16.35" width="0.3048" layer="2"/>
+<wire x1="9.55" y1="16.35" x2="9.25" y2="16.55" width="0.3048" layer="2"/>
+<wire x1="9.25" y1="16.55" x2="8.85" y2="16.55" width="0.3048" layer="2"/>
+<wire x1="8.85" y1="16.55" x2="8.6" y2="16.8" width="0.3048" layer="2"/>
+<wire x1="8.6" y1="16.8" x2="8.6" y2="17.35" width="0.3048" layer="2"/>
+<wire x1="8.6" y1="17.35" x2="8.4" y2="17.55" width="0.3048" layer="2"/>
+<wire x1="8.4" y1="17.55" x2="7.75" y2="17.55" width="0.3048" layer="2"/>
+<wire x1="7.75" y1="17.55" x2="7.4" y2="17.95" width="0.3048" layer="2"/>
+<wire x1="7.4" y1="17.95" x2="7.4" y2="26.75" width="0.3048" layer="2"/>
 <wire x1="7.4" y1="26.75" x2="7.25" y2="26.9" width="0.3048" layer="2"/>
 <wire x1="7.25" y1="26.9" x2="7.1" y2="26.9" width="0.3048" layer="2"/>
 <via x="7.1" y="26.9" extent="1-16" drill="0.25"/>
 <wire x1="7.1" y1="26.9" x2="7.3" y2="26.9" width="0.15" layer="16"/>
-<wire x1="7.3" y1="26.9" x2="7.45" y2="26.75" width="0.15" layer="16"/>
-<wire x1="7.45" y1="26.75" x2="7.8" y2="26.75" width="0.15" layer="16"/>
-<wire x1="7.8" y1="26.75" x2="8.05" y2="26.5" width="0.15" layer="16"/>
-<wire x1="8.05" y1="26.5" x2="8.05" y2="25.55" width="0.15" layer="16"/>
-<wire x1="8.05" y1="25.55" x2="8.2" y2="25.4" width="0.15" layer="16"/>
-<wire x1="8.2" y1="25.4" x2="9.2" y2="25.4" width="0.15" layer="16"/>
+<wire x1="7.3" y1="26.9" x2="7.55" y2="26.7" width="0.15" layer="16"/>
+<wire x1="7.55" y1="26.7" x2="7.55" y2="25.6" width="0.15" layer="16"/>
+<wire x1="7.55" y1="25.6" x2="7.75" y2="25.4" width="0.15" layer="16"/>
+<wire x1="7.75" y1="25.4" x2="9.2" y2="25.4" width="0.15" layer="16"/>
 <wire x1="9.2" y1="25.4" x2="9.21" y2="25.41" width="0.15" layer="16"/>
 </signal>
