File: PCB/ostc_v2/ostc_v2.brd (EAGLE design)
At the start: 31.5 x 54.8 mm, 13 parts, among them U1 ICO-640-SGG, U2 XC9536XL-10CSG48I, U3 IS62C256AL-45TLI, U4 LP5912Q3.3DRVRQ1, X1 505567-0651, X2 505567-0251, X3 150-10-640-00-001000

Commit message: Updated PCB
Routing:
- net N$19: track 30.2 -> 31.0 mm
- net N$37: track 31.1 -> 30.4 mm
- net N$41: track 28.8 -> 28.2 mm
- net N$50: track 13.3 -> 12.7 mm
- net +3.3V: track 71.0 -> 71.5 mm
Other:
- board text added: "External Turbo Switch"
- board text removed: "External Switch"

Commit message: Updated PCB
Routing:
- net N$58: track 69.7 -> 70.2 mm
