File: PCB/ostc_v2/ostc_v2.sch (EAGLE design)
At the start: 13 parts, among them IC3 150-10-640-00-001000, U1 ICO-640-SGG, U2 XC9536XL-10CSG48I, U3 IS62C256AL-45TLI, U4 LP5912Q3.3DRVRQ1, X1 505567-0651

Commit message: Modified schematics & boards
Parts:
- added X2: 505567-0251, con-molex:53261-02
- renumbered IC3 to X3
Connections:
- new net N$47: U2.PB01/11, U3G$1.A13
- new net N$48: U2.GTS2/PB01/04, U3G$1.A14
- new net N$49: U2.PB01/10, U3G$1.!OE
- new net N$50: U2.PB01/09, U3G$1.!CE
- new net N$51: U2.PB01/12, U3G$1.!WE
- net GND: now also X2-2.S
- net N$45: now also X2-1.S
Other:
- moved on the sheet: C1, C2, C3, C4, R1, R2, S1, U1, U2, U3P, U4, X1-1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

Commit message: Updated PCB files
Parts:
- removed R2: 2k, resistor:R-EU_R0805
- R1: value 4k -> 4k7
Connections:
- removed net N$46: R2.1, S1.2
- net GND: now also S1.2, X2-1.S; no longer R2.2, X2-2.S
- net N$45: now also X2-2.S; no longer X2-1.S
Other:
- moved on the sheet: X2-1, X2-2
Changed lines of the file:
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@@
 <part name="X1" library="con-molex" deviceset="53?-06" device="261" value="505567-0651"/>
 <part name="SUPPLY17" library="supply2" deviceset="+3.3V" device="" value="+3.3V"/>
-<part name="R1" library="resistor" deviceset="R-EU_" device="R0805" value="4k"/>
-<part name="R2" library="resistor" deviceset="R-EU_" device="R0805" value="2k"/>
+<part name="R1" library="resistor" deviceset="R-EU_" device="R0805" value="4k7"/>
 <part name="SUPPLY18" library="supply2" deviceset="+3.3V" device="" value="+3.3V"/>
 <part name="SUPPLY19" library="supply2" deviceset="GND" device=""/>
@@
 <instance part="SUPPLY17" gate="G$1" x="68.58" y="-142.24"/>
 <instance part="R1" gate="G$1" x="129.54" y="-142.24" rot="R90"/>
-<instance part="R2" gate="G$1" x="119.38" y="-142.24" rot="R90"/>
 <instance part="SUPPLY18" gate="G$1" x="129.54" y="-152.4" rot="R180"/>
 <instance part="SUPPLY19" gate="GND" x="119.38" y="-121.92" rot="R180"/>
@@
 <instance part="C4" gate="G$1" x="238.76" y="-76.2"/>
 <instance part="S1" gate="G$1" x="106.68" y="-142.24" rot="R90"/>
-<instance part="X2" gate="-1" x="124.46" y="-101.6"/>
-<instance part="X2" gate="-2" x="124.46" y="-104.14"/>
-<instance part="SUPPLY20" gate="GND" x="119.38" y="-109.22"/>
+<instance part="X2" gate="-1" x="124.46" y="-106.68"/>
+<instance part="X2" gate="-2" x="124.46" y="-109.22"/>
+<instance part="SUPPLY20" gate="GND" x="119.38" y="-99.06" rot="R180"/>
 </instances>
 <busses>
@@
 <segment>
 <pinref part="SUPPLY19" gate="GND" pin="GND"/>
-<pinref part="R2" gate="G$1" pin="2"/>
 <wire x1="119.38" y1="-124.46" x2="119.38" y2="-129.54" width="0.1524" layer="91"/>
-<wire x1="119.38" y1="-129.54" x2="119.38" y2="-137.16" width="0.1524" layer="91"/>
 <wire x1="104.14" y1="-129.54" x2="119.38" y2="-129.54" width="0.1524" layer="91"/>
 <junction x="119.38" y="-129.54"/>
 <pinref part="S1" gate="G$1" pin="1"/>
 <wire x1="104.14" y1="-129.54" x2="104.14" y2="-132.08" width="0.1524" layer="91"/>
-</segment>
-<segment>
-<pinref part="X2" gate="-2" pin="S"/>
+<wire x1="106.68" y1="-152.4" x2="106.68" y2="-157.48" width="0.1524" layer="91"/>
+<wire x1="106.68" y1="-157.48" x2="119.38" y2="-157.48" width="0.1524" layer="91"/>
+<pinref part="S1" gate="G$1" pin="2"/>
+<wire x1="119.38" y1="-129.54" x2="119.38" y2="-157.48" width="0.1524" layer="91"/>
+</segment>
+<segment>
+<pinref part="X2" gate="-1" pin="S"/>
 <pinref part="SUPPLY20" gate="GND" pin="GND"/>
-<wire x1="121.92" y1="-104.14" x2="119.38" y2="-104.14" width="0.1524" layer="91"/>
-<wire x1="119.38" y1="-104.14" x2="119.38" y2="-106.68" width="0.1524" layer="91"/>
+<wire x1="121.92" y1="-106.68" x2="119.38" y2="-106.68" width="0.1524" layer="91"/>
+<wire x1="119.38" y1="-106.68" x2="119.38" y2="-101.6" width="0.1524" layer="91"/>
 </segment>
 </net>
@@
 <wire x1="109.22" y1="-127" x2="129.54" y2="-127" width="0.1524" layer="91"/>
 <wire x1="129.54" y1="-127" x2="129.54" y2="-137.16" width="0.1524" layer="91"/>
-<wire x1="106.68" y1="-50.8" x2="106.68" y2="-101.6" width="0.1524" layer="91"/>
+<wire x1="106.68" y1="-50.8" x2="106.68" y2="-109.22" width="0.1524" layer="91"/>
 <pinref part="S1" gate="G$1" pin="3"/>
-<wire x1="106.68" y1="-101.6" x2="106.68" y2="-127" width="0.1524" layer="91"/>
+<wire x1="106.68" y1="-109.22" x2="106.68" y2="-127" width="0.1524" layer="91"/>
 <wire x1="109.22" y1="-132.08" x2="109.22" y2="-127" width="0.1524" layer="91"/>
 <junction x="109.22" y="-127"/>
-<pinref part="X2" gate="-1" pin="S"/>
-<wire x1="121.92" y1="-101.6" x2="106.68" y2="-101.6" width="0.1524" layer="91"/>
-<junction x="106.68" y="-101.6"/>
-</segment>
-</net>
-<net name="N$46" class="0">
-<segment>
-<wire x1="106.68" y1="-152.4" x2="106.68" y2="-157.48" width="0.1524" layer="91"/>
-<pinref part="R2" gate="G$1" pin="1"/>
-<wire x1="106.68" y1="-157.48" x2="119.38" y2="-157.48" width="0.1524" layer="91"/>
-<wire x1="119.38" y1="-157.48" x2="119.38" y2="-147.32" width="0.1524" layer="91"/>
-<pinref part="S1" gate="G$1" pin="2"/>
-</segment>
-</net>
+<pinref part="X2" gate="-2" pin="S"/>
+<wire x1="121.92" y1="-109.22" x2="106.68" y2="-109.22" width="0.1524" layer="91"/>
+<junction x="106.68" y="-109.22"/>
+</segment>
+</net>

Commit message: Updated PCBs, schematics, renders & gerbers
Parts:
- U1: device 6502:6502 -> 6502:6502SAMTEC_ICO_S
- X1: value 505567-0651 -> 5055670651; device con-molex:53261-06 -> con-molex:5055670651
- X2: value 505567-0251 -> 5055670251; device con-molex:53261-02 -> con-molex:5055670251
Connections:
- net +3.3V: now also X1.1; no longer X1-1.S
- net GND: now also X1.2, X1.7, X1.8, X2.1, X2.3, X2.4; no longer X1-2.S, X2-1.S
- net N$45: now also X2.2; no longer X2-2.S
- net N$55: now also X1.6; no longer X1-6.S
- net N$56: now also X1.5; no longer X1-5.S
- net N$57: now also X1.4; no longer X1-4.S
- net N$58: now also X1.3; no longer X1-3.S
Other:
- moved on the sheet: U1, U3P
Changed lines of the file:
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@@
 </classes>
 <parts>
-<part name="U1" library="6502" deviceset="6502" device="" value="ICO-640-SGG"/>
+<part name="U1" library="6502" deviceset="6502" device="SAMTEC_ICO_S" value="ICO-640-SGG"/>
 <part name="X3" library="DIL-header" deviceset="DIL40" device="" value="150-10-640-00-001000"/>
 <part name="U2" library="xilinx-xc9" deviceset="CX9536_CS48" device="" value="XC9536XL-10CSG48I"/>
@@
 <part name="SUPPLY15" library="supply2" deviceset="GND" device=""/>
 <part name="SUPPLY16" library="supply2" deviceset="GND" device=""/>
-<part name="X1" library="con-molex" deviceset="53?-06" device="261" value="505567-0651"/>
 <part name="SUPPLY17" library="supply2" deviceset="+3.3V" device="" value="+3.3V"/>
 <part name="R1" library="resistor" deviceset="R-EU_" device="R0805" value="4k7"/>
@@
 <part name="C4" library="resistor" deviceset="C-EU" device="C1206K" value="100n"/>
 <part name="S1" library="SS312SAH4-R" deviceset="SS312SAH4-R" device=""/>
-<part name="X2" library="con-molex" deviceset="53?-02" device="261" value="505567-0251"/>
 <part name="SUPPLY20" library="supply2" deviceset="GND" device=""/>
+<part name="X2" library="con-molex" deviceset="5055670251" device=""/>
+<part name="X1" library="con-molex" deviceset="5055670651" device=""/>
+<part name="SUPPLY21" library="supply2" deviceset="GND" device=""/>
+<part name="SUPPLY22" library="supply2" deviceset="GND" device=""/>
 </parts>
 <sheets>
@@
 <instance part="SUPPLY15" gate="GND" x="152.4" y="60.96"/>
 <instance part="SUPPLY16" gate="GND" x="17.78" y="81.28" rot="R180"/>
-<instance part="X1" gate="-1" x="73.66" y="-149.86"/>
-<instance part="X1" gate="-2" x="73.66" y="-152.4"/>
-<instance part="X1" gate="-3" x="73.66" y="-154.94"/>
-<instance part="X1" gate="-4" x="73.66" y="-157.48"/>
-<instance part="X1" gate="-5" x="73.66" y="-160.02"/>
-<instance part="X1" gate="-6" x="73.66" y="-162.56"/>
 <instance part="SUPPLY17" gate="G$1" x="68.58" y="-142.24"/>
 <instance part="R1" gate="G$1" x="129.54" y="-142.24" rot="R90"/>
@@
 <instance part="C4" gate="G$1" x="238.76" y="-76.2"/>
 <instance part="S1" gate="G$1" x="106.68" y="-142.24" rot="R90"/>
-<instance part="X2" gate="-1" x="124.46" y="-106.68"/>
-<instance part="X2" gate="-2" x="124.46" y="-109.22"/>
 <instance part="SUPPLY20" gate="GND" x="119.38" y="-99.06" rot="R180"/>
+<instance part="X2" gate="A" x="127" y="-106.68"/>
+<instance part="X1" gate="A" x="76.2" y="-149.86"/>
+<instance part="SUPPLY21" gate="GND" x="76.2" y="-172.72"/>
+<instance part="SUPPLY22" gate="GND" x="127" y="-119.38"/>
 </instances>
 <busses>
@@
 <junction x="66.04" y="-129.54"/>
 <wire x1="63.5" y1="-129.54" x2="63.5" y2="-152.4" width="0.1524" layer="91"/>
-<pinref part="X1" gate="-2" pin="S"/>
-<wire x1="63.5" y1="-152.4" x2="71.12" y2="-152.4" width="0.1524" layer="91"/>
+<wire x1="63.5" y1="-152.4" x2="76.2" y2="-152.4" width="0.1524" layer="91"/>
 <junction x="63.5" y="-129.54"/>
+<pinref part="X1" gate="A" pin="2"/>
 </segment>
 <segment>
@@
 </segment>
 <segment>
-<pinref part="X2" gate="-1" pin="S"/>
 <pinref part="SUPPLY20" gate="GND" pin="GND"/>
-<wire x1="121.92" y1="-106.68" x2="119.38" y2="-106.68" width="0.1524" layer="91"/>
 <wire x1="119.38" y1="-106.68" x2="119.38" y2="-101.6" width="0.1524" layer="91"/>
+<pinref part="X2" gate="A" pin="1"/>
+<wire x1="127" y1="-106.68" x2="119.38" y2="-106.68" width="0.1524" layer="91"/>
+</segment>
+<segment>
+<pinref part="X1" gate="A" pin="7"/>
+<pinref part="X1" gate="A" pin="8"/>
+<wire x1="76.2" y1="-165.1" x2="76.2" y2="-167.64" width="0.1524" layer="91"/>
+<pinref part="SUPPLY21" gate="GND" pin="GND"/>
+<wire x1="76.2" y1="-167.64" x2="76.2" y2="-170.18" width="0.1524" layer="91"/>
+<junction x="76.2" y="-167.64"/>
+</segment>
+<segment>
+<pinref part="X2" gate="A" pin="3"/>
+<pinref part="X2" gate="A" pin="4"/>
+<wire x1="127" y1="-111.76" x2="127" y2="-114.3" width="0.1524" layer="91"/>
+<pinref part="SUPPLY22" gate="GND" pin="GND"/>
+<wire x1="127" y1="-114.3" x2="127" y2="-116.84" width="0.1524" layer="91"/>
+<junction x="127" y="-114.3"/>
 </segment>
 </net>
@@
 <pinref part="SUPPLY17" gate="G$1" pin="+3.3V"/>
 <wire x1="68.58" y1="-144.78" x2="68.58" y2="-149.86" width="0.1524" layer="91"/>
-<pinref part="X1" gate="-1" pin="S"/>
-<wire x1="68.58" y1="-149.86" x2="71.12" y2="-149.86" width="0.1524" layer="91"/>
+<pinref part="X1" gate="A" pin="1"/>
+<wire x1="76.2" y1="-149.86" x2="68.58" y2="-149.86" width="0.1524" layer="91"/>
 </segment>
 <segment>
@@
 <net name="N$55" class="0">
 <segment>
-<pinref part="X1" gate="-6" pin="S"/>
 <pinref part="U2" gate="G$1" pin="TMS"/>
-<wire x1="71.12" y1="-162.56" x2="60.96" y2="-162.56" width="0.1524" layer="91"/>
+<wire x1="76.2" y1="-162.56" x2="60.96" y2="-162.56" width="0.1524" layer="91"/>
 <wire x1="60.96" y1="-162.56" x2="60.96" y2="-124.46" width="0.1524" layer="91"/>
+<pinref part="X1" gate="A" pin="6"/>
 </segment>
 </net>
@@
 <pinref part="U2" gate="G$1" pin="TDI"/>
 <wire x1="55.88" y1="-124.46" x2="55.88" y2="-160.02" width="0.1524" layer="91"/>
-<pinref part="X1" gate="-5" pin="S"/>
-<wire x1="55.88" y1="-160.02" x2="71.12" y2="-160.02" width="0.1524" layer="91"/>
+<wire x1="55.88" y1="-160.02" x2="76.2" y2="-160.02" width="0.1524" layer="91"/>
+<pinref part="X1" gate="A" pin="5"/>
 </segment>
 </net>
@@
 <pinref part="U2" gate="G$1" pin="TDO"/>
 <wire x1="58.42" y1="-124.46" x2="58.42" y2="-157.48" width="0.1524" layer="91"/>
-<pinref part="X1" gate="-4" pin="S"/>
-<wire x1="58.42" y1="-157.48" x2="71.12" y2="-157.48" width="0.1524" layer="91"/>
+<wire x1="58.42" y1="-157.48" x2="76.2" y2="-157.48" width="0.1524" layer="91"/>
+<pinref part="X1" gate="A" pin="4"/>
 </segment>
 </net>
@@
 <pinref part="U2" gate="G$1" pin="TCK"/>
 <wire x1="53.34" y1="-124.46" x2="53.34" y2="-154.94" width="0.1524" layer="91"/>
-<pinref part="X1" gate="-3" pin="S"/>
-<wire x1="53.34" y1="-154.94" x2="71.12" y2="-154.94" width="0.1524" layer="91"/>
+<wire x1="53.34" y1="-154.94" x2="76.2" y2="-154.94" width="0.1524" layer="91"/>
+<pinref part="X1" gate="A" pin="3"/>
 </segment>
 </net>
@@
 <wire x1="109.22" y1="-132.08" x2="109.22" y2="-127" width="0.1524" layer="91"/>
 <junction x="109.22" y="-127"/>
-<pinref part="X2" gate="-2" pin="S"/>
-<wire x1="121.92" y1="-109.22" x2="106.68" y2="-109.22" width="0.1524" layer="91"/>
+<wire x1="127" y1="-109.22" x2="106.68" y2="-109.22" width="0.1524" layer="91"/>
 <junction x="106.68" y="-109.22"/>
-</segment>
-</net>
+<pinref part="X2" gate="A" pin="2"/>
+</segment>
+</net>

Commit message: Updated PCBs, schematics, gerbers & renders
Connections:
- net GND: now also S1.4, S1.5
Changed lines of the file:
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@@
 <wire x1="106.68" y1="-157.48" x2="119.38" y2="-157.48" width="0.1524" layer="91"/>
 <pinref part="S1" gate="G$1" pin="2"/>
-<wire x1="119.38" y1="-129.54" x2="119.38" y2="-157.48" width="0.1524" layer="91"/>
+<wire x1="119.38" y1="-129.54" x2="119.38" y2="-142.24" width="0.1524" layer="91"/>
+<pinref part="S1" gate="G$1" pin="4"/>
+<wire x1="119.38" y1="-142.24" x2="119.38" y2="-144.78" width="0.1524" layer="91"/>
+<wire x1="119.38" y1="-144.78" x2="119.38" y2="-157.48" width="0.1524" layer="91"/>
+<wire x1="116.84" y1="-142.24" x2="119.38" y2="-142.24" width="0.1524" layer="91"/>
+<pinref part="S1" gate="G$1" pin="5"/>
+<wire x1="116.84" y1="-144.78" x2="119.38" y2="-144.78" width="0.1524" layer="91"/>
+<junction x="119.38" y="-142.24"/>
+<junction x="119.38" y="-144.78"/>
 </segment>
 <segment>
