File: PCB/ostc_v3/ostc_v3.sch (EAGLE design)
At the start: 18 parts, among them IC3 150-10-640-00-001000, U1 ICO-640-SGG, U2 XC9536XL-10CSG48I, U3 IS62C256AL-45TLI, U4 LP5912Q3.3DRVRQ1, U5 MAX4996ETG, U6 MAX4996ETG, U7 MAX4996ETG, U8 MAX4996ETG, X1 505567-0651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

Commit message: Corrected schematic#
Connections:
- new net N$77: U2.PB01/11, U3G$1.A13
- new net N$78: U2.GTS2/PB01/04, U3G$1.A14
- new net N$79: U2.PB01/10, U3G$1.!OE
- new net N$80: U2.PB01/09, U3G$1.!CE
- new net N$81: U2.PB01/12, U3G$1.!WE
Changed lines of the file:
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@@
 <setting verticaltext="up"/>
 </settings>
-<grid distance="1" unitdist="mm" unit="mm" style="lines" multiple="1" display="no" altdistance="0.1" altunitdist="mm" altunit="mm"/>
+<grid distance="0.1" unitdist="inch" unit="inch" style="lines" multiple="1" display="no" altdistance="0.05" altunitdist="inch" altunit="inch"/>
 <layers>
 <layer number="1" name="Top" color="4" fill="1" visible="yes" active="no"/>
@@
 <segment>
 <pinref part="U2" gate="G$1" pin="PB01/06"/>
-<wire x1="53.34" y1="-287.02" x2="53.34" y2="-279.4" width="0.1524" layer="91"/>
-<wire x1="53.34" y1="-279.4" x2="106.68" y2="-279.4" width="0.1524" layer="91"/>
+<wire x1="53.34" y1="-287.02" x2="53.34" y2="-281.94" width="0.1524" layer="91"/>
+<wire x1="53.34" y1="-281.94" x2="106.68" y2="-281.94" width="0.1524" layer="91"/>
 <pinref part="R1" gate="G$1" pin="2"/>
 <wire x1="106.68" y1="-358.14" x2="129.54" y2="-358.14" width="0.1524" layer="91"/>
 <wire x1="129.54" y1="-358.14" x2="129.54" y2="-365.76" width="0.1524" layer="91"/>
 <wire x1="129.54" y1="-365.76" x2="129.54" y2="-368.3" width="0.1524" layer="91"/>
-<wire x1="106.68" y1="-279.4" x2="106.68" y2="-358.14" width="0.1524" layer="91"/>
+<wire x1="106.68" y1="-281.94" x2="106.68" y2="-358.14" width="0.1524" layer="91"/>
 <pinref part="S1" gate="G$1" pin="NO_2"/>
 <wire x1="121.92" y1="-365.76" x2="129.54" y2="-365.76" width="0.1524" layer="91"/>
@@
 </segment>
 </net>
+<net name="N$77" class="0">
+<segment>
+<pinref part="U3" gate="G$1" pin="A13"/>
+<pinref part="U2" gate="G$1" pin="PB01/11"/>
+<wire x1="220.98" y1="40.64" x2="193.04" y2="40.64" width="0.1524" layer="91"/>
+<wire x1="193.04" y1="40.64" x2="193.04" y2="15.24" width="0.1524" layer="91"/>
+<wire x1="193.04" y1="15.24" x2="187.96" y2="15.24" width="0.1524" layer="91"/>
+<wire x1="187.96" y1="15.24" x2="187.96" y2="-185.42" width="0.1524" layer="91"/>
+<wire x1="187.96" y1="-185.42" x2="172.72" y2="-185.42" width="0.1524" layer="91"/>
+<wire x1="172.72" y1="-185.42" x2="172.72" y2="-269.24" width="0.1524" layer="91"/>
+<wire x1="172.72" y1="-269.24" x2="66.04" y2="-269.24" width="0.1524" layer="91"/>
+<wire x1="66.04" y1="-269.24" x2="66.04" y2="-287.02" width="0.1524" layer="91"/>
+</segment>
+</net>
+<net name="N$78" class="0">
+<segment>
+<pinref part="U2" gate="G$1" pin="GTS2/PB01/04"/>
+<wire x1="48.26" y1="-287.02" x2="48.26" y2="-279.4" width="0.1524" layer="91"/>
+<wire x1="48.26" y1="-279.4" x2="55.88" y2="-279.4" width="0.1524" layer="91"/>
+<wire x1="55.88" y1="-279.4" x2="55.88" y2="-276.86" width="0.1524" layer="91"/>
+<wire x1="55.88" y1="-276.86" x2="68.58" y2="-276.86" width="0.1524" layer="91"/>
+<wire x1="68.58" y1="-276.86" x2="68.58" y2="-271.78" width="0.1524" layer="91"/>
+<wire x1="68.58" y1="-271.78" x2="175.26" y2="-271.78" width="0.1524" layer="91"/>
+<wire x1="175.26" y1="-271.78" x2="175.26" y2="-187.96" width="0.1524" layer="91"/>
+<wire x1="175.26" y1="-187.96" x2="190.5" y2="-187.96" width="0.1524" layer="91"/>
+<wire x1="190.5" y1="-187.96" x2="190.5" y2="12.7" width="0.1524" layer="91"/>
+<wire x1="190.5" y1="12.7" x2="195.58" y2="12.7" width="0.1524" layer="91"/>
+<wire x1="195.58" y1="12.7" x2="195.58" y2="38.1" width="0.1524" layer="91"/>
+<pinref part="U3" gate="G$1" pin="A14"/>
+<wire x1="195.58" y1="38.1" x2="220.98" y2="38.1" width="0.1524" layer="91"/>
+</segment>
+</net>
+<net name="N$79" class="0">
+<segment>
+<pinref part="U2" gate="G$1" pin="PB01/10"/>
+<wire x1="63.5" y1="-287.02" x2="63.5" y2="-279.4" width="0.1524" layer="91"/>
+<wire x1="63.5" y1="-279.4" x2="71.12" y2="-279.4" width="0.1524" layer="91"/>
+<wire x1="71.12" y1="-279.4" x2="71.12" y2="-274.32" width="0.1524" layer="91"/>
+<wire x1="71.12" y1="-274.32" x2="177.8" y2="-274.32" width="0.1524" layer="91"/>
+<wire x1="177.8" y1="-274.32" x2="177.8" y2="-190.5" width="0.1524" layer="91"/>
+<wire x1="177.8" y1="-190.5" x2="193.04" y2="-190.5" width="0.1524" layer="91"/>
+<wire x1="193.04" y1="-190.5" x2="193.04" y2="10.16" width="0.1524" layer="91"/>
+<wire x1="193.04" y1="10.16" x2="198.12" y2="10.16" width="0.1524" layer="91"/>
+<wire x1="198.12" y1="10.16" x2="198.12" y2="33.02" width="0.1524" layer="91"/>
+<pinref part="U3" gate="G$1" pin="!OE"/>
+<wire x1="198.12" y1="33.02" x2="220.98" y2="33.02" width="0.1524" layer="91"/>
+</segment>
+</net>
+<net name="N$80" class="0">
+<segment>
+<pinref part="U2" gate="G$1" pin="PB01/09"/>
+<wire x1="60.96" y1="-287.02" x2="60.96" y2="-284.48" width="0.1524" layer="91"/>
+<wire x1="60.96" y1="-284.48" x2="73.66" y2="-284.48" width="0.1524" layer="91"/>
+<wire x1="73.66" y1="-284.48" x2="73.66" y2="-276.86" width="0.1524" layer="91"/>
+<wire x1="73.66" y1="-276.86" x2="180.34" y2="-276.86" width="0.1524" layer="91"/>
+<wire x1="180.34" y1="-276.86" x2="180.34" y2="-193.04" width="0.1524" layer="91"/>
+<wire x1="180.34" y1="-193.04" x2="195.58" y2="-193.04" width="0.1524" layer="91"/>
+<wire x1="195.58" y1="-193.04" x2="195.58" y2="7.62" width="0.1524" layer="91"/>
+<wire x1="195.58" y1="7.62" x2="200.66" y2="7.62" width="0.1524" layer="91"/>
+<wire x1="200.66" y1="7.62" x2="200.66" y2="30.48" width="0.1524" layer="91"/>
+<pinref part="U3" gate="G$1" pin="!CE"/>
+<wire x1="200.66" y1="30.48" x2="220.98" y2="30.48" width="0.1524" layer="91"/>
+</segment>
+</net>
+<net name="N$81" class="0">
+<segment>
+<pinref part="U2" gate="G$1" pin="PB01/12"/>
+<wire x1="86.36" y1="-307.34" x2="104.14" y2="-307.34" width="0.1524" layer="91"/>
+<wire x1="104.14" y1="-307.34" x2="104.14" y2="-279.4" width="0.1524" layer="91"/>
+<wire x1="104.14" y1="-279.4" x2="182.88" y2="-279.4" width="0.1524" layer="91"/>
+<wire x1="182.88" y1="-279.4" x2="182.88" y2="-195.58" width="0.1524" layer="91"/>
+<wire x1="182.88" y1="-195.58" x2="203.2" y2="-195.58" width="0.1524" layer="91"/>
+<wire x1="203.2" y1="-195.58" x2="203.2" y2="25.4" width="0.1524" layer="91"/>
+<pinref part="U3" gate="G$1" pin="!WE"/>
+<wire x1="203.2" y1="25.4" x2="220.98" y2="25.4" width="0.1524" layer="91"/>
+</segment>
+</net>

Commit message: Updated PCB
Parts:
- renumbered IC3 to X3

Commit message: Updated PCBs, schematics, renders & gerbers
Parts:
- added X4: 150-10-640-00-001000, DIL-header:DIL40
- C1, C2, C3, C4: device resistor:C-EUC1206K -> resistor:C-EUC0805
- U1: device 6502:6502 -> 6502:6502SAMTEC_ICO_C
- X1: device con-molex:53261-06 -> con-molex:5055670651
- X3: value 150-10-640-00-001000 -> 5055670251; device DIL-header:DIL40 -> con-molex:5055670251
Connections:
- net +3.3V: now also X1.1; no longer X1-1.S
- net +5V: now also S1.MP1, S1.MP2, X4.8; no longer X3.8
- net GND: now also X1.2, X1.7, X1.8, X3.2, X3.3, X3.4, X4.1, X4.21, X4.35, X4.36, X4.5; no longer S1.MP1, S1.MP2, X1-2.S, X3.1, X3.21, X3.35, X3.36, X3.5
- net N$1: now also X4.2; no longer X3.2
- net N$10: now also X4.13; no longer X3.13
- net N$11: now also X4.14; no longer X3.14
- net N$12: now also X4.15; no longer X3.15
- net N$13: now also X4.16; no longer X3.16
- net N$14: now also X4.17; no longer X3.17
- net N$15: now also X4.18; no longer X3.18
- net N$16: now also X4.19; no longer X3.19
- net N$17: now also X4.20; no longer X3.20
- net N$19: now also X4.22; no longer X3.22
- net N$2: now also X4.3; no longer X3.3
- net N$20: now also X4.23; no longer X3.23
- net N$3: now also X4.4; no longer X3.4
- net N$31: now also X4.37; no longer X3.37
- net N$32: now also X4.38; no longer X3.38
- net N$33: now also X4.39; no longer X3.39
- net N$34: now also X4.40; no longer X3.40
- net N$4: now also X4.6; no longer X3.6
- net N$45: now also X3.1
- net N$48: now also X4.25; no longer X3.25
- net N$5: now also X4.7; no longer X3.7
- net N$50: now also X4.26; no longer X3.26
- net N$52: now also X4.27; no longer X3.27
- net N$55: now also X1.6; no longer X1-6.S
- net N$56: now also X1.5; no longer X1-5.S
- net N$57: now also X1.4; no longer X1-4.S
- net N$58: now also X1.3; no longer X1-3.S
- net N$6: now also X4.9; no longer X3.9
- net N$60: now also X4.24; no longer X3.24
- net N$61: now also X4.28; no longer X3.28
- net N$63: now also X4.31; no longer X3.31
- net N$65: now also X4.29; no longer X3.29
- net N$66: now also X4.30; no longer X3.30
- net N$69: now also X4.32; no longer X3.32
- net N$7: now also X4.10; no longer X3.10
- net N$72: now also X4.33; no longer X3.33
- net N$73: now also X4.34; no longer X3.34
- net N$8: now also X4.11; no longer X3.11
- net N$9: now also X4.12; no longer X3.12
Other:
- moved on the sheet: X2
