File: PCB/ostc_v3/ostc_v3.brd (EAGLE design)
At the start: 31.5 x 54.2 mm, 19 parts, among them U1 ICO-640-SGG, U2 XC9536XL-10CSG48I, U3 IS62C256AL-45TLI, U4 LP5912Q3.3DRVRQ1, U5 MAX4996ETG, U6 MAX4996ETG, U7 MAX4996ETG, U8 MAX4996ETG, X1 505567-0651, X2 5055670251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

Commit message: Updated v3 PCB
Routing:
- net N$57: track 11.3 -> 88.1 mm, vias 0 -> 3
- net N$45: track 28.9 -> 73.2 mm, vias 2 -> 3
- net N$66: track 0.00 -> 28.2 mm, vias 0 -> 2
- net N$51: track 29.6 -> 52.0 mm, vias 2 -> 5
- net N$63: track 0.00 -> 20.2 mm, vias 0 -> 1
- net N$41: track 0.00 -> 11.8 mm, vias 0 -> 1
- net N$78: track 7.71 -> 19.0 mm, vias 0 -> 2
- net N$42: track 0.08 -> 8.16 mm, vias 0 -> 2
- net GND: track 17.6 -> 12.3 mm, vias 23 -> 22
- net N$39: track 7.83 -> 12.0 mm, vias 0 -> 1
- net N$76: track 15.9 -> 16.5 mm
- net N$68: vias 2 -> 1
